File: Pi1541io.sch (KiCad schematic (older format))
At the start: 55 parts, among them J1 IEC1, J10 SDA, J11 SCL, J12 I2C, J13 SDA, J14 SDA, J15 SDA, J2 IEC2, J3 IEC3, J4 ExtSpkr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

Commit message: Added an additional solder bridge that is now needed to connect the SRQ line from the bus. This closes #1.
Parts:
- added J16: GS2, Connectors:GS2, symbol conn:GS2
Connections:
- wire segments 179 -> 183
Other:
- moved on the sheet: J9, Q5, R14, R15
Changed lines of the file:
@@
 L Transistor:BSS138 Q5
 U 1 1 5B084802
-P 4550 6350
-F 0 "Q5" V 4800 6350 50  0000 C CNN
-F 1 "BSS138" V 4891 6350 50  0000 C CNN
-F 2 "TO_SOT_Packages_SMD:SOT-23" H 4750 6275 50  0001 L CIN
-F 3 "https://www.fairchildsemi.com/datasheets/BS/BSS138.pdf" H 4550 6350 50  0001 L CNN
-	1    4550 6350
+P 4550 6250
+F 0 "Q5" V 4800 6250 50  0000 C CNN
+F 1 "BSS138" V 4891 6250 50  0000 C CNN
+F 2 "TO_SOT_Packages_SMD:SOT-23" H 4750 6175 50  0001 L CIN
+F 3 "https://www.fairchildsemi.com/datasheets/BS/BSS138.pdf" H 4550 6250 50  0001 L CNN
+	1    4550 6250
 	0    1    1    0
 $EndComp
@@
 L device:R R14
 U 1 1 5B084809
-P 4250 6300
-F 0 "R14" H 4320 6346 50  0000 L CNN
-F 1 "10k" H 4320 6255 50  0000 L CNN
-F 2 "Resistors_SMD:R_0805" V 4180 6300 50  0001 C CNN
-F 3 "" H 4250 6300 50  0001 C CNN
-	1    4250 6300
-	1    0    0    -1
-$EndComp
-Wire Wire Line
-	4250 6150 4550 6150
-Wire Wire Line
-	4350 6450 4250 6450
+P 4250 6200
+F 0 "R14" H 4320 6246 50  0000 L CNN
+F 1 "10k" H 4320 6155 50  0000 L CNN
+F 2 "Resistors_SMD:R_0805" V 4180 6200 50  0001 C CNN
+F 3 "" H 4250 6200 50  0001 C CNN
+	1    4250 6200
+	1    0    0    -1
+$EndComp
+Wire Wire Line
+	4250 6050 4550 6050
+Wire Wire Line
+	4350 6350 4250 6350
 $Comp
 L power:+3.3V #PWR0121
 U 1 1 5B084812
-P 4250 6150
-F 0 "#PWR0121" H 4250 6000 50  0001 C CNN
-F 1 "+3.3V" H 4250 6290 50  0000 C CNN
-F 2 "" H 4250 6150 50  0000 C CNN
-F 3 "" H 4250 6150 50  0000 C CNN
-	1    4250 6150
-	1    0    0    -1
-$EndComp
-Connection ~ 4250 6150
+P 4250 6050
+F 0 "#PWR0121" H 4250 5900 50  0001 C CNN
+F 1 "+3.3V" H 4250 6190 50  0000 C CNN
+F 2 "" H 4250 6050 50  0000 C CNN
+F 3 "" H 4250 6050 50  0000 C CNN
+	1    4250 6050
+	1    0    0    -1
+$EndComp
+Connection ~ 4250 6050
 $Comp
 L device:R R15
 U 1 1 5B084819
-P 4750 6300
-F 0 "R15" H 4820 6346 50  0000 L CNN
-F 1 "10k" H 4820 6255 50  0000 L CNN
-F 2 "Resistors_SMD:R_0805" V 4680 6300 50  0001 C CNN
-F 3 "" H 4750 6300 50  0001 C CNN
-	1    4750 6300
+P 4750 6200
+F 0 "R15" H 4820 6246 50  0000 L CNN
+F 1 "10k" H 4820 6155 50  0000 L CNN
+F 2 "Resistors_SMD:R_0805" V 4680 6200 50  0001 C CNN
+F 3 "" H 4750 6200 50  0001 C CNN
+	1    4750 6200
 	1    0    0    -1
 $EndComp
@@
 L power:+5V #PWR0122
 U 1 1 5B084820
-P 4750 6150
-F 0 "#PWR0122" H 4750 6000 50  0001 C CNN
-F 1 "+5V" H 4750 6290 50  0000 C CNN
-F 2 "" H 4750 6150 50  0000 C CNN
-F 3 "" H 4750 6150 50  0000 C CNN
-	1    4750 6150
-	1    0    0    -1
-$EndComp
-Wire Wire Line
-	4250 6450 4150 6450
-Connection ~ 4250 6450
-Wire Wire Line
-	4750 6450 4850 6450
-Connection ~ 4750 6450
-Text GLabel 4850 6450 2    50   Input ~ 0
+P 4750 6050
+F 0 "#PWR0122" H 4750 5900 50  0001 C CNN
+F 1 "+5V" H 4750 6190 50  0000 C CNN
+F 2 "" H 4750 6050 50  0000 C CNN
+F 3 "" H 4750 6050 50  0000 C CNN
+	1    4750 6050
+	1    0    0    -1
+$EndComp
+Wire Wire Line
+	4250 6350 4150 6350
+Connection ~ 4250 6350
+Connection ~ 4750 6350
+Text GLabel 5550 5950 2    50   Input ~ 0
 SRQ
-Text GLabel 4150 6450 0    50   Input ~ 0
+Text GLabel 4150 6350 0    50   Input ~ 0
 SRQ_3V
-Text GLabel 3500 6500 0    50   Input ~ 0
+Text GLabel 3500 6400 0    50   Input ~ 0
 SRQ_BD
 $Comp
 L conn:GS3 J9
 U 1 1 5B09227D
-P 3650 6600
-F 0 "J9" H 3650 6905 50  0000 C CNN
-F 1 "GS3" H 3650 6814 50  0000 C CNN
-F 2 "Connectors:GS3" V 3738 6526 50  0001 C CNN
-F 3 "" H 3650 6600 50  0001 C CNN
-	1    3650 6600
-	1    0    0    -1
-$EndComp
-Text GLabel 3500 6700 0    50   Input ~ 0
+P 3650 6500
+F 0 "J9" H 3650 6805 50  0000 C CNN
+F 1 "GS3" H 3650 6714 50  0000 C CNN
+F 2 "Connectors:GS3" V 3738 6426 50  0001 C CNN
+F 3 "" H 3650 6500 50  0001 C CNN
+	1    3650 6500
+	1    0    0    -1
+$EndComp
+Text GLabel 3500 6600 0    50   Input ~ 0
 SRQ_IN
-Text GLabel 3800 6600 2    50   Input ~ 0
+Text GLabel 3800 6500 2    50   Input ~ 0
 SRQ_3V
 $Comp
@@
 Text GLabel 1350 6550 0    50   Input ~ 0
 SRQ_BD
-Text GLabel 2650 6550 2    50   Input ~ 0
-SRQ
 Wire Wire Line
 	2450 6550 2500 6550
@@
 	1050 2750 900  2750
 Wire Notes Line
-	5300 5950 950  5950
-Wire Notes Line
-	950  5950 950  6950
-Wire Notes Line
-	950  6950 5300 6950
-Wire Notes Line
-	5300 6950 5300 5950
-Text Notes 4000 6900 0    50   ~ 0
+	5800 5850 950  5850
+Wire Notes Line
+	950  5850 950  7000
+Wire Notes Line
+	950  7000 5800 7000
+Wire Notes Line
+	5800 7000 5800 5850
+Text Notes 4000 6950 0    50   ~ 0
 Reserved SRQ support (optional)
 Wire Notes Line
@@
 	1450 2750 3500 2750
 Connection ~ 1050 2750
+$Comp
+L conn:GS2 J16
+U 1 1 5BCF72C0
+P 5350 6150
+F 0 "J16" H 5418 6196 50  0000 L CNN
+F 1 "GS2" H 5418 6105 50  0000 L CNN
+F 2 "Connectors:GS2" V 5424 6150 50  0001 C CNN
+F 3 "" H 5350 6150 50  0001 C CNN
+	1    5350 6150
+	1    0    0    -1
+$EndComp
+Wire Wire Line
+	5550 5950 5350 5950
+Wire Wire Line
+	4750 6350 5350 6350
+Wire Wire Line
+	5350 6350 5350 6750
+Wire Wire Line
+	5350 6750 2650 6750
+Wire Wire Line
+	2650 6750 2650 6550
+Connection ~ 5350 6350
 $EndSCHEMATC
